Commit message: update jaka s5 moveit config

File: hugmi_description/urdf/jaka_s5.urdf (robot description, URDF)
Before this commit: robot jaka_s5, 8 links, 7 joints
Links:
- removed link Link_0
- removed link Link_1
- removed link Link_2
- removed link Link_3
- removed link Link_4
- removed link Link_5
- removed link Link_6
- added link link_0, mass 0.52663; collision mesh filename=package://hugmi_description/meshes/jaka_s5_meshes/link_0.STL; visual mesh filename=package://hugmi_description/meshes/jaka_s5_meshes/link_0.STL
- added link link_1, mass 15.135; collision mesh filename=package://hugmi_description/meshes/jaka_s5_meshes/link_1.STL; visual mesh filename=package://hugmi_description/meshes/jaka_s5_meshes/link_1.STL
- added link link_2, mass 45.847; collision mesh filename=package://hugmi_description/meshes/jaka_s5_meshes/link_2.STL; visual mesh filename=package://hugmi_description/meshes/jaka_s5_meshes/link_2.STL
- added link link_3, mass 18.05; collision mesh filename=package://hugmi_description/meshes/jaka_s5_meshes/link_3.STL; visual mesh filename=package://hugmi_description/meshes/jaka_s5_meshes/link_3.STL
- added link link_4, mass 5.5377; collision mesh filename=package://hugmi_description/meshes/jaka_s5_meshes/link_4.STL; visual mesh filename=package://hugmi_description/meshes/jaka_s5_meshes/link_4.STL
- added link link_5, mass 6.3339; collision mesh filename=package://hugmi_description/meshes/jaka_s5_meshes/link_5.STL; visual mesh filename=package://hugmi_description/meshes/jaka_s5_meshes/link_5.STL
- added link link_6, mass 0.23261; collision mesh filename=package://hugmi_description/meshes/jaka_s5_meshes/link_6.STL; visual mesh filename=package://hugmi_description/meshes/jaka_s5_meshes/link_6.STL
Joints:
- removed joint Joint1
- removed joint Joint2
- removed joint Joint3
- removed joint Joint4
- removed joint Joint5
- removed joint Joint6
- removed joint fixed
- added joint base_joint: type fixed, parent world, child link_0
- added joint joint1: type revolute, parent link_0, child link_1, origin xyz=0 -0.00022535 0.12015 rpy=0 0 0, axis 0 0 -1, limit lower=-6.28 upper=6.28 effort=2000 velocity=1.57
- added joint joint2: type revolute, parent link_1, child link_2, origin xyz=0 0 0 rpy=1.5708 0 0, axis 0 0 1, limit lower=-1.48 upper=4.62 effort=5000 velocity=1.57
- added joint joint3: type revolute, parent link_2, child link_3, origin xyz=0.43 0 0 rpy=0 0 0, axis 0 0 1, limit lower=-3.05 upper=3.05 effort=5000 velocity=1.57
- added joint joint4: type revolute, parent link_3, child link_4, origin xyz=0.3685 0 -0.114 rpy=0 0 0, axis 0 0 1, limit lower=-1.48 upper=4.62 effort=2000 velocity=1.57
- added joint joint5: type revolute, parent link_4, child link_5, origin xyz=0 -0.1135 0 rpy=1.5708 0 0, axis 0 0 1, limit lower=-6.28 upper=6.28 effort=3000 velocity=1.57
- added joint joint6: type revolute, parent link_5, child link_6, origin xyz=0.00026137 0.1175 0.00025782 rpy=-1.5708 0 0, axis 0 0 1, limit lower=-6.28 upper=6.28 effort=1000 velocity=1.57

File: jaka_s5_moveit_config/config/jaka_s5.ros2_control.xacro (robot description, xacro)
@@ -8,43 +8,43 @@
                 <plugin>mock_components/GenericSystem</plugin>
             </hardware>
-            <joint name="Joint1">
+            <joint name="joint1">
                 <command_interface name="position"/>
                 <state_interface name="position">
-                  <param name="initial_value">${initial_positions['Joint1']}</param>
+                  <param name="initial_value">${initial_positions['joint1']}</param>
                 </state_interface>
                 <state_interface name="velocity"/>
             </joint>
-            <joint name="Joint2">
+            <joint name="joint2">
                 <command_interface name="position"/>
                 <state_interface name="position">
-                  <param name="initial_value">${initial_positions['Joint2']}</param>
+                  <param name="initial_value">${initial_positions['joint2']}</param>
                 </state_interface>
                 <state_interface name="velocity"/>
             </joint>
-            <joint name="Joint3">
+            <joint name="joint3">
                 <command_interface name="position"/>
                 <state_interface name="position">
-                  <param name="initial_value">${initial_positions['Joint3']}</param>
+                  <param name="initial_value">${initial_positions['joint3']}</param>
                 </state_interface>
                 <state_interface name="velocity"/>
             </joint>
-            <joint name="Joint4">
+            <joint name="joint4">
                 <command_interface name="position"/>
                 <state_interface name="position">
-                  <param name="initial_value">${initial_positions['Joint4']}</param>
+                  <param name="initial_value">${initial_positions['joint4']}</param>
                 </state_interface>
                 <state_interface name="velocity"/>
             </joint>
-            <joint name="Joint5">
+            <joint name="joint5">
                 <command_interface name="position"/>
                 <state_interface name="position">
-                  <param name="initial_value">${initial_positions['Joint5']}</param>
+                  <param name="initial_value">${initial_positions['joint5']}</param>
                 </state_interface>
                 <state_interface name="velocity"/>
             </joint>
-            <joint name="Joint6">
+            <joint name="joint6">
                 <command_interface name="position"/>
                 <state_interface name="position">
-                  <param name="initial_value">${initial_positions['Joint6']}</param>
+                  <param name="initial_value">${initial_positions['joint6']}</param>
                 </state_interface>
                 <state_interface name="velocity"/>
