Commit message: add robotiq 85 gripper urdf and update moveit config

File: hugmi_description/urdf/hugmi.ros2_control.xacro (robot description, xacro)
@@ -2,5 +2,5 @@
 <robot xmlns:xacro="http://www.ros.org/wiki/xacro">
     <xacro:macro name="hugmi_ros2_control" params="name initial_positions_file">
-        <xacro:property name="initial_positions" value="${load_yaml(initial_positions_file)['initial_positions']}"/>
+        <xacro:property name="initial_positions" value="${xacro.load_yaml(initial_positions_file)['initial_positions']}"/>
         <ros2_control name="${name}" type="system">
             <hardware>

File: hugmi_description/urdf/hugmi.urdf.xacro (robot description, xacro)
@@ -5,29 +5,15 @@
     <xacro:arg name="right_arm_initial_positions_file"
         default="$(find hugmi_description)/config/right_initial_positions.yaml"/>
+    <!-- Xacro imports -->
+    <xacro:include filename="$(find hugmi_description)/urdf/jaka_s5_arm_macro.xacro" />
+    <xacro:include filename="$(find hugmi_description)/urdf/robotiq_85_gripper.urdf.xacro"/>
+    <xacro:include filename="$(find hugmi_description)/urdf/hugmi_body.urdf.xacro"/>
+    <xacro:include filename="$(find hugmi_description)/urdf/robotiq_85_gripper.urdf.xacro" />
+    <link name="world"/>
     <!-- body link -->
-    <link name="body">
-        <inertial>
-            <origin xyz="0.0028167 -0.00019454 0.019544" rpy="0 0 0" />
-            <mass value="0.52663" />
-            <inertia ixx="0.0006297" ixy="6.7091E-08" ixz="3.4682E-06" iyy="0.00095727" iyz="2.4476E-07" izz="0.0014514" />
-        </inertial>
-        <visual>
-            <origin xyz="0 0 0" rpy="0 0 0" />
-            <geometry>
-                <mesh filename="package://hugmi_description/meshes/body_meshes/body_simplified.stl" />
-            </geometry>
-            <material name="">
-                <color rgba="0.79216 0.81961 0.93333 1" />
-            </material>
-        </visual>
-        <collision>
-            <origin xyz="0 0 0" rpy="0 0 0" />
-            <geometry>
-                <mesh filename="package://hugmi_description/meshes/body_meshes/body_simplified.stl" />
-            </geometry>
-        </collision>
-    </link>
-    <!-- Xacro imports -->
-    <xacro:include filename="jaka_s5_arm_macro.xacro" />
+    <xacro:hugmi_body
+        parent="world">
+        <origin xyz="0 0 0" rpy="0 0 0" />
+    </xacro:hugmi_body>
     <!-- Left arm -->
     <xacro:jaka_s5_arm
@@ -38,4 +24,9 @@
         <origin xyz="0.232 0.284 0.816" rpy="1.888 0.594 1.753" />
     </xacro:jaka_s5_arm>
+    <xacro:robotiq_85_gripper
+        prefix="left_"
+        parent="left_link_6">
+        <origin xyz="0 0 0" rpy="0 -1.571 0"/>
+    </xacro:robotiq_85_gripper>
     <!-- Right arm -->
     <xacro:jaka_s5_arm
@@ -44,5 +35,10 @@
         parent="body"
         initial_positions_file="$(arg right_arm_initial_positions_file)">
-        <origin xyz="-0.233 0.284 0.818" rpy="-1.888 0.594  1.389" />
+        <origin xyz="-0.233 0.284 0.818" rpy="-1.888 0.594 1.389" />
     </xacro:jaka_s5_arm>
+    <xacro:robotiq_85_gripper
+        prefix="right_"
+        parent="right_link_6">
+        <origin xyz="0 0 0" rpy="0 -1.571 0"/>
+    </xacro:robotiq_85_gripper>
 </robot>

File: hugmi_description/urdf/jaka_s5_arm_macro.xacro (robot description, xacro)
@@ -4,4 +4,5 @@
         <!-- ros2_control -->
         <xacro:include filename="$(find hugmi_description)/urdf/jaka_s5_arm.ros2_control.xacro" />
+        <xacro:include filename="$(find hugmi_description)/urdf/jaka_s5_arm.transmission.xacro" />
         <xacro:jaka_s5_arm_ros2_control name="${name}" initial_positions_file="${initial_positions_file}" prefix="${prefix}"/>
         <!-- base_joint fixes base_link to the environment-->
@@ -207,69 +208,5 @@
             <limit lower="-6.28" upper="6.28" effort="1000" velocity="1.57" />
         </joint>
-        <transmission name="${prefix}trans_joint1">
-            <type>transmission_interface/SimpleTransmission</type>
-            <joint name="${prefix}joint1">
-                <hardwareInterface>hardware_interface/PositionJointInterface</hardwareInterface>
-            </joint>
-            <actuator name="${prefix}joint1_motor">
-                <hardwareInterface>hardware_interface/PositionJointInterface</hardwareInterface>
-                <mechanicalReduction>1</mechanicalReduction>
-            </actuator>
-        </transmission>
-        <transmission name="${prefix}trans_joint2">
-            <type>transmission_interface/SimpleTransmission</type>
-            <joint name="${prefix}joint2">
-                <hardwareInterface>hardware_interface/PositionJointInterface</hardwareInterface>
-            </joint>
-            <actuator name="${prefix}joint2_motor">
-                <hardwareInterface>hardware_interface/PositionJointInterface</hardwareInterface>
-                <mechanicalReduction>1</mechanicalReduction>
-            </actuator>
-        </transmission>
-        <transmission name="${prefix}trans_joint3">
-            <type>transmission_interface/SimpleTransmission</type>
-            <joint name="${prefix}joint3">
-                <hardwareInterface>hardware_interface/PositionJointInterface</hardwareInterface>
-            </joint>
-            <actuator name="${prefix}joint3_motor">
-                <hardwareInterface>hardware_interface/PositionJointInterface</hardwareInterface>
-                <mechanicalReduction>1</mechanicalReduction>
-            </actuator>
-        </transmission>
-        <transmission name="${prefix}trans_joint4">
-            <type>transmission_interface/SimpleTransmission</type>
-            <joint name="${prefix}joint4">
-                <hardwareInterface>hardware_interface/PositionJointInterface</hardwareInterface>
-            </joint>
-            <actuator name="${prefix}joint4_motor">
-                <hardwareInterface>hardware_interface/PositionJointInterface</hardwareInterface>
-                <mechanicalReduction>1</mechanicalReduction>
-            </actuator>
-        </transmission>
-        <transmission name="${prefix}trans_joint5">
-            <type>transmission_interface/SimpleTransmission</type>
-            <joint name="${prefix}joint5">
-                <hardwareInterface>hardware_interface/PositionJointInterface</hardwareInterface>
-            </joint>
-            <actuator name="${prefix}joint5_motor">
-                <hardwareInterface>hardware_interface/PositionJointInterface</hardwareInterface>
-                <mechanicalReduction>1</mechanicalReduction>
-            </actuator>
-        </transmission>
-        <transmission name="${prefix}trans_joint6">
-            <type>transmission_interface/SimpleTransmission</type>
-            <joint name="${prefix}joint6">
-                <hardwareInterface>hardware_interface/PositionJointInterface</hardwareInterface>
-            </joint>
-            <actuator name="${prefix}joint6_motor">
-                <hardwareInterface>hardware_interface/PositionJointInterface</hardwareInterface>
-                <mechanicalReduction>1</mechanicalReduction>
-            </actuator>
-        </transmission>
-        <gazebo>
-            <plugin name="gazebo_ros_control" filename="libgazebo_ros_control.so">
-                <robotNamespace>/</robotNamespace>
-            </plugin>
-        </gazebo>
+    <xacro:jaka_s5_arm_transmission prefix="${prefix}" />
     </xacro:macro>
 </robot>

File: hugmi_moveit_config/config/hugmi.ros2_control.xacro (robot description, xacro)
@@ -2,5 +2,5 @@
 <robot xmlns:xacro="http://www.ros.org/wiki/xacro">
     <xacro:macro name="hugmi_ros2_control" params="name initial_positions_file">
-        <xacro:property name="initial_positions" value="${load_yaml(initial_positions_file)['initial_positions']}"/>
+        <xacro:property name="initial_positions" value="${xacro.load_yaml(initial_positions_file)['initial_positions']}"/>
         <ros2_control name="${name}" type="system">
             <hardware>
@@ -92,4 +92,18 @@
                 <state_interface name="velocity"/>
             </joint>
+            <joint name="left_robotiq_85_left_knuckle_joint">
+                <command_interface name="position"/>
+                <state_interface name="position">
+                  <param name="initial_value">${initial_positions['left_robotiq_85_left_knuckle_joint']}</param>
+                </state_interface>
+                <state_interface name="velocity"/>
+            </joint>
+            <joint name="right_robotiq_85_left_knuckle_joint">
+                <command_interface name="position"/>
+                <state_interface name="position">
+                  <param name="initial_value">${initial_positions['right_robotiq_85_left_knuckle_joint']}</param>
+                </state_interface>
+                <state_interface name="velocity"/>
+            </joint>
         </ros2_control>
     </xacro:macro>
